File: vco_4046/vco_4046.sch (KiCad schematic (older format))
At the start: 15 parts, among them J1 Conn_01x02_Male, J2 Conn_02x05_Odd_Even, J3 Conn_01x02_Male, J4 Conn_01x02_Male, J5 Conn_01x03_Male, U1 4046, U2 LM358

Commit message: 4046 VCO PCB
Parts:
- C1, C4, C5: footprint (none) -> Capacitor_THT:C_Disc_D5.0mm_W2.5mm_P5.00mm
- C2, C3: footprint (none) -> Capacitor_THT:CP_Radial_D5.0mm_P2.00mm
- J1, J3, J4: footprint (none) -> Connector_PinHeader_2.54mm:PinHeader_1x02_P2.54mm_Vertical
- J2: footprint (none) -> Connector_IDC:IDC-Header_2x05_P2.54mm_Vertical
- J5: footprint (none) -> Connector_PinHeader_2.54mm:PinHeader_1x03_P2.54mm_Vertical
- R1, R2: footprint (none) -> Resistor_THT:R_Axial_DIN0207_L6.3mm_D2.5mm_P10.16mm_Horizontal
- RV1: footprint (none) -> Potentiometer_THT:Potentiometer_ACP_CA9-V10_Vertical
- U1: footprint (none) -> Package_DIP:DIP-16_W7.62mm_LongPads
- U2: footprint (none) -> Package_DIP:DIP-8_W7.62mm_LongPads
Changed lines of the file:
@@
 F 0 "U1" H 4950 4550 50  0000 C CNN
 F 1 "4046" H 5000 4450 50  0000 C CNN
-F 2 "" H 4850 3900 50  0001 C CNN
+F 2 "Package_DIP:DIP-16_W7.62mm_LongPads" H 4850 3900 50  0001 C CNN
 F 3 "https://assets.nexperia.com/documents/data-sheet/HEF4046B.pdf" H 4850 3900 50  0001 C CNN
 	1    4850 3900
@@
 F 0 "C1" H 4092 3896 50  0000 L CNN
 F 1 "10n" H 4092 3805 50  0000 L CNN
-F 2 "" H 4000 3850 50  0001 C CNN
+F 2 "Capacitor_THT:C_Disc_D5.0mm_W2.5mm_P5.00mm" H 4000 3850 50  0001 C CNN
 F 3 "~" H 4000 3850 50  0001 C CNN
 	1    4000 3850
@@
 F 0 "C3" H 5488 2446 50  0000 L CNN
 F 1 "10u" H 5488 2355 50  0000 L CNN
-F 2 "" H 5400 2400 50  0001 C CNN
+F 2 "Capacitor_THT:CP_Radial_D5.0mm_P2.00mm" H 5400 2400 50  0001 C CNN
 F 3 "~" H 5400 2400 50  0001 C CNN
 	1    5400 2400
@@
 F 0 "R1" H 4070 4346 50  0000 L CNN
 F 1 "100k" H 4070 4255 50  0000 L CNN
-F 2 "" V 3930 4300 50  0001 C CNN
+F 2 "Resistor_THT:R_Axial_DIN0207_L6.3mm_D2.5mm_P10.16mm_Horizontal" V 3930 4300 50  0001 C CNN
 F 3 "~" H 4000 4300 50  0001 C CNN
 	1    4000 4300
@@
 F 0 "U2" H 6200 4433 50  0000 C CNN
 F 1 "LM358" H 6200 4524 50  0000 C CNN
-F 2 "" H 6200 4800 50  0001 C CNN
+F 2 "Package_DIP:DIP-8_W7.62mm_LongPads" H 6200 4800 50  0001 C CNN
 F 3 "http://www.ti.com/lit/ds/symlink/lm2904-n.pdf" H 6200 4800 50  0001 C CNN
 	1    6200 4800
@@
 F 0 "U2" H 6308 2296 50  0000 L CNN
 F 1 "LM358" H 6308 2205 50  0000 L CNN
-F 2 "" H 6350 2250 50  0001 C CNN
+F 2 "Package_DIP:DIP-8_W7.62mm_LongPads" H 6350 2250 50  0001 C CNN
 F 3 "http://www.ti.com/lit/ds/symlink/lm2904-n.pdf" H 6350 2250 50  0001 C CNN
 	3    6350 2250
@@
 F 0 "J1" H 3408 4189 50  0000 C CNN
 F 1 "Conn_01x02_Male" H 3408 4190 50  0001 C CNN
-F 2 "" H 3300 4100 50  0001 C CNN
+F 2 "Connector_PinHeader_2.54mm:PinHeader_1x02_P2.54mm_Vertical" H 3300 4100 50  0001 C CNN
 F 3 "~" H 3300 4100 50  0001 C CNN
 	1    3300 4100
@@
 F 0 "U2" H 7000 4533 50  0000 C CNN
 F 1 "LM358" H 7000 4624 50  0000 C CNN
-F 2 "" H 7000 4900 50  0001 C CNN
+F 2 "Package_DIP:DIP-8_W7.62mm_LongPads" H 7000 4900 50  0001 C CNN
 F 3 "http://www.ti.com/lit/ds/symlink/lm2904-n.pdf" H 7000 4900 50  0001 C CNN
 	2    7000 4900
@@
 F 0 "J5" H 8272 4778 50  0000 R CNN
 F 1 "Conn_01x03_Male" H 8272 4733 50  0001 R CNN
-F 2 "" H 8300 4800 50  0001 C CNN
+F 2 "Connector_PinHeader_2.54mm:PinHeader_1x03_P2.54mm_Vertical" H 8300 4800 50  0001 C CNN
 F 3 "~" H 8300 4800 50  0001 C CNN
 	1    8300 4800
@@
 F 0 "J4" H 8272 3978 50  0000 R CNN
 F 1 "Conn_01x02_Male" H 8272 3933 50  0001 R CNN
-F 2 "" H 8300 4050 50  0001 C CNN
+F 2 "Connector_PinHeader_2.54mm:PinHeader_1x02_P2.54mm_Vertical" H 8300 4050 50  0001 C CNN
 F 3 "~" H 8300 4050 50  0001 C CNN
 	1    8300 4050
@@
 F 0 "R2" H 7720 4346 50  0000 L CNN
 F 1 "100k" H 7720 4255 50  0000 L CNN
-F 2 "" V 7580 4300 50  0001 C CNN
+F 2 "Resistor_THT:R_Axial_DIN0207_L6.3mm_D2.5mm_P10.16mm_Horizontal" V 7580 4300 50  0001 C CNN
 F 3 "~" H 7650 4300 50  0001 C CNN
 	1    7650 4300
@@
 F 0 "RV1" V 7250 4250 50  0000 C CNN
 F 1 "10k" V 7150 4250 50  0000 C CNN
-F 2 "" H 7000 4350 50  0001 C CNN
+F 2 "Potentiometer_THT:Potentiometer_ACP_CA9-V10_Vertical" H 7000 4350 50  0001 C CNN
 F 3 "~" H 7000 4350 50  0001 C CNN
 	1    7000 4350
@@
 F 0 "J3" H 6272 3428 50  0000 R CNN
 F 1 "Conn_01x02_Male" H 6272 3383 50  0001 R CNN
-F 2 "" H 6300 3500 50  0001 C CNN
+F 2 "Connector_PinHeader_2.54mm:PinHeader_1x02_P2.54mm_Vertical" H 6300 3500 50  0001 C CNN
 F 3 "~" H 6300 3500 50  0001 C CNN
 	1    6300 3500
@@
 F 0 "J2" H 4850 2550 50  0000 C CNN
 F 1 "Conn_02x05_Odd_Even" H 4850 2576 50  0001 C CNN
-F 2 "" H 4800 2250 50  0001 C CNN
+F 2 "Connector_IDC:IDC-Header_2x05_P2.54mm_Vertical" H 4800 2250 50  0001 C CNN
 F 3 "~" H 4800 2250 50  0001 C CNN
 	1    4800 2250
@@
 F 0 "C2" H 5488 2146 50  0000 L CNN
 F 1 "10u" H 5488 2055 50  0000 L CNN
-F 2 "" H 5400 2100 50  0001 C CNN
+F 2 "Capacitor_THT:CP_Radial_D5.0mm_P2.00mm" H 5400 2100 50  0001 C CNN
 F 3 "~" H 5400 2100 50  0001 C CNN
 	1    5400 2100
@@
 F 0 "C4" H 5792 2146 50  0000 L CNN
 F 1 "100n" H 5792 2055 50  0000 L CNN
-F 2 "" H 5700 2100 50  0001 C CNN
+F 2 "Capacitor_THT:C_Disc_D5.0mm_W2.5mm_P5.00mm" H 5700 2100 50  0001 C CNN
 F 3 "~" H 5700 2100 50  0001 C CNN
 	1    5700 2100
@@
 F 0 "C5" H 5792 2446 50  0000 L CNN
 F 1 "100n" H 5792 2355 50  0000 L CNN
-F 2 "" H 5700 2400 50  0001 C CNN
+F 2 "Capacitor_THT:C_Disc_D5.0mm_W2.5mm_P5.00mm" H 5700 2400 50  0001 C CNN
 F 3 "~" H 5700 2400 50  0001 C CNN
 	1    5700 2400
